Commit message: replaced decimated stl files with originals

File: rover_urdf/urdf/MR24-DT-A00.00_2.SLDASM.urdf (robot description, URDF)
Before this commit: robot MR24-DT-A00.00_2.SLDASM, 7 links, 6 joints
Links:
- removed link Front_right Wheel
- added link Front_Right Wheel, mass 1.45375895562017; collision mesh filename=../meshes/Front_Right Wheel.STL; visual mesh filename=../meshes/Front_Right Wheel.STL
Joints:
- joint Front_Right Wheel Joint: child Front_right Wheel -> Front_Right Wheel

Commit message: wip

File: rover_urdf/urdf/MR24-DT-A00.00_2.SLDASM.urdf (robot description, URDF)
Before this commit: robot MR24-DT-A00.00_2.SLDASM, 7 links, 6 joints
Links:
- removed link Front_right Wheel
- added link Front_Right Wheel, mass 1.45375895562017; collision mesh filename=../meshes/Front_Right Wheel.STL; visual mesh filename=../meshes/Front_Right Wheel.STL
Joints:
- joint Center_Left Wheel Joint: origin xyz=0 0 0 rpy=0 0 0 -> xyz=0.000000 0.005589 0.506384 rpy=0 0 0
- joint Center_Right Wheel Joint: origin xyz=0 0 0 rpy=0 0 0 -> xyz=0.000000 0.005563 0.506384 rpy=0 0 0
- joint Front_Left Wheel Joint: origin xyz=0 0 0 rpy=0 0 0 -> xyz=0.000000 0.000000 0.498351 rpy=0 0 0
- joint Front_Right Wheel Joint: child Front_right Wheel -> Front_Right Wheel; origin xyz=0 0 0 rpy=0 0 0 -> xyz=0.000000 0.000000 0.498464 rpy=0 0 0
- joint Rear_Left Wheel Joint: origin xyz=0 0 0 rpy=0 0 0 -> xyz=0.000000 0.000000 0.490124 rpy=0 0 0
- joint Rear_Right Wheel Joint: origin xyz=0 0 0 rpy=0 0 0 -> xyz=0.000000 0.000000 0.489950 rpy=0 0 0

File: src/gazebo/launch/robot.urdf (robot description, URDF)
Before this commit: robot robot, 4 links, 0 joints
Links:
- link robot/caster: geometry visual sphere radius=0.1
- link robot/chassis: geometry visual mesh filename=package://gazebo/launch/rover_base_link.STL scale=2.0 2.0 2.0
- link robot/left_wheel: geometry visual mesh filename=package://gazebo/launch/rover_wheel.STL scale=2.0 2.0 2.0
- link robot/right_wheel: geometry visual mesh filename=package://gazebo/launch/rover_wheel.STL scale=2.0 2.0 2.0
