Commit message: compressed stl meshes, visually replaced current robot with uwrt urdf

File: src/gazebo/launch/robot.urdf (robot description, URDF)
Before this commit: robot robot, 4 links, 0 joints
Links:
- added link robot/front_left_wheel_visual; visual mesh filename=package://gazebo/launch/rover_front_left_wheel.stl
- added link robot/front_right_wheel_visual; visual mesh filename=package://gazebo/launch/rover_front_right_wheel.stl
- added link robot/rear_left_wheel_visual; visual mesh filename=package://gazebo/launch/rover_rear_left_wheel.stl
- added link robot/rear_right_wheel_visual; visual mesh filename=package://gazebo/launch/rover_rear_right_wheel.stl
- link robot/caster: geometry visual sphere radius=0.01
- link robot/chassis: geometry visual mesh filename=package://gazebo/launch/rover_base_link.stl
- link robot/left_wheel: geometry visual mesh filename=package://gazebo/launch/rover_center_left_wheel.stl
- link robot/right_wheel: geometry visual mesh filename=package://gazebo/launch/rover_center_right_wheel.stl
Joints:
- added joint front_left_wheel_visual_joint: type fixed, parent robot/chassis, child robot/front_left_wheel_visual, origin xyz=0.404 0.6 0 rpy=-1.5707 0 0
- added joint front_right_wheel_visual_joint: type fixed, parent robot/chassis, child robot/front_right_wheel_visual, origin xyz=0.404 -0.6 0 rpy=-1.5707 0 0
- added joint rear_left_wheel_visual_joint: type fixed, parent robot/chassis, child robot/rear_left_wheel_visual, origin xyz=-0.398 0.6 0 rpy=-1.5707 0 0
- added joint rear_right_wheel_visual_joint: type fixed, parent robot/chassis, child robot/rear_right_wheel_visual, origin xyz=-0.398 -0.6 0 rpy=-1.5707 0 0

Commit message: made urdf refer to branch instead of master

File: src/gazebo/launch/robot.urdf (robot description, URDF)
Before this commit: robot robot, 8 links, 4 joints
Links:
- link robot/chassis: geometry visual mesh filename=https://raw.githubusercontent.com/WATonomous/wato_rover/add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
- link robot/front_left_wheel_visual: geometry visual mesh filename=https://raw.githubusercontent.com/WATonomous/wato_rover/add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
- link robot/front_right_wheel_visual: geometry visual mesh filename=https://raw.githubusercontent.com/WATonomous/wato_rover/add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
- link robot/left_wheel: geometry visual mesh filename=https://raw.githubusercontent.com/WATonomous/wato_rover/add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
- link robot/rear_left_wheel_visual: geometry visual mesh filename=https://raw.githubusercontent.com/WATonomous/wato_rover/add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
- link robot/rear_right_wheel_visual: geometry visual mesh filename=https://raw.githubusercontent.com/WATonomous/wato_rover/add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
- link robot/right_wheel: geometry visual mesh filename=https://raw.githubusercontent.com/WATonomous/wato_rover/add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

Commit message: moved wheel locations

File: src/gazebo/launch/robot.urdf (robot description, URDF)
Before this commit: robot robot, 8 links, 4 joints
Joints:
- joint front_left_wheel_visual_joint: origin xyz=0.404 0.6 0 rpy=-1.5707 0 0 -> xyz=0 0 0 rpy=0 0 0
- joint front_right_wheel_visual_joint: origin xyz=0.404 -0.6 0 rpy=-1.5707 0 0 -> xyz=0 0 0 rpy=0 0 0
- joint rear_left_wheel_visual_joint: origin xyz=-0.398 0.6 0 rpy=-1.5707 0 0 -> xyz=0 0 0 rpy=0 0 0
- joint rear_right_wheel_visual_joint: origin xyz=-0.398 -0.6 0 rpy=-1.5707 0 0 -> xyz=0 0 0 rpy=0 0 0

Commit message: moved wheel positions

File: src/gazebo/launch/robot.urdf (robot description, URDF)
Before this commit: robot robot, 8 links, 4 joints
Joints:
- added joint left_wheel_joint: type fixed, parent robot/chassis, child robot/left_wheel, origin xyz=-0.5 0.6 0 rpy=-1.5707 0 0
- added joint right_wheel_joint: type fixed, parent robot/chassis, child robot/right_wheel, origin xyz=-0.5 -0.6 0 rpy=-1.5707 0 0

Commit message: edited rotation

File: src/gazebo/launch/robot.urdf (robot description, URDF)
Before this commit: robot robot, 8 links, 6 joints
Joints:
- joint front_left_wheel_visual_joint: origin xyz=0 0 0 rpy=0 0 0 -> xyz=0.40398 0.43855 0.0080468 rpy=0 0 0
- joint front_right_wheel_visual_joint: origin xyz=0 0 0 rpy=0 0 0 -> xyz=0.40398 -0.43855 0.0080468 rpy=0 0 0
- joint left_wheel_joint: origin xyz=-0.5 0.6 0 rpy=-1.5707 0 0 -> xyz=0 0.48455 0 rpy=-1.5707 0 0
- joint rear_left_wheel_visual_joint: origin xyz=0 0 0 rpy=0 0 0 -> xyz=-0.39807 0.48455 0.016315 rpy=0 0 0
- joint rear_right_wheel_visual_joint: origin xyz=0 0 0 rpy=0 0 0 -> xyz=-0.39807 -0.48455 0.016315 rpy=0 0 0
- joint right_wheel_joint: origin xyz=-0.5 -0.6 0 rpy=-1.5707 0 0 -> xyz=0 -0.48455 0 rpy=-1.5707 0 0

Commit message: wip

File: src/gazebo/launch/robot.urdf (robot description, URDF)
Before this commit: robot robot, 8 links, 6 joints
Links:
- removed link robot/caster

Commit message: moved around origin of stl files

File: src/gazebo/launch/robot.urdf (robot description, URDF)
Before this commit: robot robot, 7 links, 6 joints
Joints:
- joint left_wheel_joint: origin xyz=0 0.48455 0 rpy=-1.5707 0 0 -> xyz=0 0.48455 0 rpy=0 0 0
- joint right_wheel_joint: origin xyz=0 -0.48455 0 rpy=-1.5707 0 0 -> xyz=0 -0.48455 0 rpy=0 0 0

Commit message: almost working

File: src/gazebo/launch/robot.urdf (robot description, URDF)
Before this commit: robot robot, 7 links, 6 joints
Links:
- link robot/chassis: geometry visual mesh filename=rover_base_link.stl
- link robot/front_left_wheel_visual: geometry visual mesh filename=rover_front_left_wheel.stl
- link robot/front_right_wheel_visual: geometry visual mesh filename=rover_front_right_wheel.stl
- link robot/left_wheel: geometry visual mesh filename=rover_center_left_wheel.stl
- link robot/rear_left_wheel_visual: geometry visual mesh filename=rover_rear_left_wheel.stl
- link robot/rear_right_wheel_visual: geometry visual mesh filename=rover_rear_right_wheel.stl
- link robot/right_wheel: geometry visual mesh filename=rover_center_right_wheel.stl

Commit message: adjusted collision of the original caster/wheels/chassis to visually match the rover

File: src/gazebo/launch/robot.urdf (robot description, URDF)
Before this commit: robot robot, 7 links, 6 joints
Links:
- removed link robot/front_left_wheel_visual
- removed link robot/front_right_wheel_visual
- removed link robot/rear_left_wheel_visual
- removed link robot/rear_right_wheel_visual
- added link robot/fl_whl; visual mesh filename=rover_front_left_wheel.stl
- added link robot/fr_whl; visual mesh filename=rover_front_right_wheel.stl
- added link robot/rl_whl; visual mesh filename=rover_rear_left_wheel.stl
- added link robot/rr_whl; visual mesh filename=rover_rear_right_wheel.stl
Joints:
- removed joint front_left_wheel_visual_joint
- removed joint front_right_wheel_visual_joint
- removed joint rear_left_wheel_visual_joint
- removed joint rear_right_wheel_visual_joint
- added joint fl_whl_joint: type fixed, parent robot/chassis, child robot/fl_whl, origin xyz=0.40398 0.43855 0.0080468 rpy=0 0 0
- added joint fr_whl_joint: type fixed, parent robot/chassis, child robot/fr_whl, origin xyz=0.40398 -0.43855 0.0080468 rpy=0 0 0
- added joint rl_whl_joint: type fixed, parent robot/chassis, child robot/rl_whl, origin xyz=-0.39807 0.48455 0.016315 rpy=0 0 0
- added joint rr_whl_joint: type fixed, parent robot/chassis, child robot/rr_whl, origin xyz=-0.39807 -0.48455 0.016315 rpy=0 0 0

Commit message: foxglove gets urdf from github url instead of local filepath

File: src/gazebo/launch/robot.urdf (robot description, URDF)
Before this commit: robot robot, 7 links, 6 joints
Links:
- link robot/chassis: geometry visual mesh filename=https://raw.githubusercontent.com/WATonomous/wato_rover/add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
- link robot/fl_whl: geometry visual mesh filename=https://raw.githubusercontent.com/WATonomous/wato_rover/add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
- link robot/fr_whl: geometry visual mesh filename=https://raw.githubusercontent.com/WATonomous/wato_rover/add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
- link robot/left_wheel: geometry visual mesh filename=https://raw.githubusercontent.com/WATonomous/wato_rover/add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
- link robot/right_wheel: geometry visual mesh filename=https://raw.githubusercontent.com/WATonomous/wato_rover/add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
- link robot/rl_whl: geometry visual mesh filename=https://raw.githubusercontent.com/WATonomous/wato_rover/add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
- link robot/rr_whl: geometry visual mesh filename=https://raw.githubusercontent.com/WATonomous/wato_rover/add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
