Commit message: add smaller boulders

File: src/gazebo/launch/mars_env.urdf (robot description, URDF)
Before this commit: robot mars_environment, 6 links, 5 joints
Links:
- link boulder1_link: geometry collision cylinder length=0.3 radius=0.5; visual cylinder length=0.3 radius=0.5
- link boulder2_link: geometry collision cylinder length=0.5 radius=0.8; visual cylinder length=0.5 radius=0.8
- link boulder3_link: geometry collision sphere radius=0.4; visual sphere radius=0.4
- link boulder4_link: geometry collision cylinder length=0.6 radius=0.6; visual cylinder length=0.6 radius=0.6
- link boulder5_link: geometry collision sphere radius=0.3; visual sphere radius=0.3

Commit message: Update Github file hosting links

File: src/gazebo/launch/mars_env.urdf (robot description, URDF)
Before this commit: robot mars_environment, 4 links, 3 joints
Links:
- link mallet: geometry collision mesh filename=https://raw.githubusercontent.com/WATonomous/wato_rover/mas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 scale=0.1 0.1 0.1; visual mesh filename=https://raw.githubusercontent.com/WATonomous/wato_rover/mas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 scale=0.1 0.1 0.1
- link water_bottle: geometry collision mesh filename=https://raw.githubusercontent.com/WATonomous/wato_rover/mas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 scale=0.1 0.1 0.1; visual mesh filename=https://raw.githubusercontent.com/WATonomous/wato_rover/mas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 scale=0.1 0.1 0.1

Commit message: Fix object detection integration by modifying onnx file and processing code

File: src/gazebo/launch/mars_env.urdf (robot description, URDF)
Before this commit: robot mars_environment, 4 links, 3 joints
Links:
- link mallet: geometry collision mesh filename=https://raw.githubusercontent.com/WATonomous/wato_rover/mas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 scale=0.4 0.4 0.4; visual mesh filename=https://raw.githubusercontent.com/WATonomous/wato_rover/mas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 scale=0.4 0.4 0.4
- link water_bottle: geometry collision mesh filename=https://raw.githubusercontent.com/WATonomous/wato_rover/mas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 scale=0.4 0.4 0.4; visual mesh filename=https://raw.githubusercontent.com/WATonomous/wato_rover/mas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 scale=0.4 0.4 0.4

Commit message: added object to simulation

File: src/gazebo/launch/mars_env.urdf (robot description, URDF)
Before this commit: robot mars_environment, 4 links, 3 joints
Links:
- added link pick; collision mesh filename=./pick.stl scale=0.004 0.004 0.004; visual mesh filename=./pick.stl scale=0.004 0.004 0.004
Joints:
- added joint pick_joint: type fixed, parent desert, child pick, origin xyz=0 1.2 -2 rpy=0 0 0

Commit message: update stl link

File: src/gazebo/launch/mars_env.urdf (robot description, URDF)
Before this commit: robot mars_environment, 5 links, 4 joints
Links:
- link desert: geometry collision mesh filename=https://raw.githubusercontent.com/WATonomous/wato_rover/dem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 scale=0.1 0.1 0.1; visual mesh filename=https://raw.githubusercontent.com/WATonomous/wato_rover/dem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 scale=0.1 0.1 0.1

Commit message: new

File: src/gazebo/launch/mars_env.urdf (robot description, URDF)
Before this commit: robot mars_environment, 5 links, 4 joints
Links:
- link desert: geometry collision mesh filename=https://raw.githubusercontent.com/WATonomous/wato_rover/mar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 scale=0.1 0.1 0.1; visual mesh filename=https://raw.githubusercontent.com/WATonomous/wato_rover/mar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 scale=0.1 0.1 0.1
